File: MysX2USB.sch (KiCad schematic (older format))
At the start: 9 parts, among them P1 USB_A, P2 MYSX_1.2, P3 supply, U1 FT230XS

Commit message: Changed to use MysX1.1, and made the pcb smaller. Added pdf of schematics
Parts:
- P2: footprint mysensors_connectors:MYSX_1.2 -> mysensors_connectors:MYSX_1.0; symbol MYSX_1.2 -> MYSX_1.0
Changed lines of the file:
@@
 Date "2016-03-20"
 Rev "0.5"
-Comp ""
-Comment1 "Thomas Mørch"
+Comp "Mysensors.org"
+Comment1 "Created by Thomas B. Mørch"
 Comment2 ""
 Comment3 ""
@@
 $EndDescr
 $Comp
-L MYSX_1.2 P2
+L MYSX_1.0 P2
 U 1 1 56E907D4
 P 6950 4100
 F 0 "P2" H 7475 4331 50  0000 C CNN
 F 1 "MYSX_1.2" H 7475 4240 50  0000 C CNN
-F 2 "mysensors_connectors:MYSX_1.2" H 6950 2900 60  0001 C CNN
+F 2 "mysensors_connectors:MYSX_1.0" H 6950 2900 60  0001 C CNN
 F 3 "" H 6950 2900 60  0000 C CNN
 	1    6950 4100
@@
 Connection ~ 4550 3150
 $Comp
-L GND #PWR08
+L GND #PWR07
 U 1 1 56E9134E
 P 4550 2750
-F 0 "#PWR08" H 4550 2500 50  0001 C CNN
+F 0 "#PWR07" H 4550 2500 50  0001 C CNN
 F 1 "GND" H 4558 2577 50  0000 C CNN
 F 2 "" H 4550 2750 50  0000 C CNN

Commit message: Updated to MysX2.0
Parts:
- added D3: V_TARGET, LEDs:LED-0603, symbol LED
- added R3: R, Resistors_SMD:R_0603_HandSoldering, symbol R
- C1: footprint Capacitors_SMD:C_0603 -> Capacitors_SMD:C_0603_HandSoldering
- D1: value LED -> RX
- D2: value LED -> TX
- P2: value MYSX_1.2 -> MYSX_2.0; symbol MYSX_1.0 -> MYSX_2.0
- R1, R2: footprint Resistors_SMD:R_0603 -> Resistors_SMD:R_0603_HandSoldering
- U1: value FT230XS -> FT231XS; footprint Housings_SSOP:SSOP-16_3.9x4.9mm_Pitch0.635mm -> Housings_SSOP:SSOP-20_4.4x6.5mm_Pitch0.65mm; symbol FT230XS -> FT231XS
Connections:
- net labels added: RST
- wire segments 24 -> 26
Changed lines of the file:
@@
 $EndDescr
 $Comp
-L MYSX_1.0 P2
+L MYSX_2.0 P2
 U 1 1 56E907D4
 P 6950 4100
 F 0 "P2" H 7475 4331 50  0000 C CNN
-F 1 "MYSX_1.2" H 7475 4240 50  0000 C CNN
+F 1 "MYSX_2.0" H 7475 4240 50  0000 C CNN
 F 2 "mysensors_connectors:MYSX_1.0" H 6950 2900 60  0001 C CNN
 F 3 "" H 6950 2900 60  0000 C CNN
@@
 $EndComp
 $Comp
-L FT230XS U1
+L FT231XS U1
 U 1 1 56E90861
-P 4850 4300
-F 0 "U1" H 4850 5178 50  0000 C CNN
-F 1 "FT230XS" H 4850 5087 50  0000 C CNN
-F 2 "Housings_SSOP:SSOP-16_3.9x4.9mm_Pitch0.635mm" H 4850 5086 50  0001 C CNN
-F 3 "" H 4850 4300 50  0000 C CNN
-	1    4850 4300
+P 4850 4500
+F 0 "U1" H 4850 5378 50  0000 C CNN
+F 1 "FT231XS" H 4850 5287 50  0000 C CNN
+F 2 "Housings_SSOP:SSOP-20_4.4x6.5mm_Pitch0.65mm" H 4850 5286 50  0001 C CNN
+F 3 "" H 4850 4500 50  0000 C CNN
+	1    4850 4500
 	1    0    0    -1
 $EndComp
@@
 	4750 3350 4750 3600
 $Comp
-L GND #PWR04
-U 1 1 56E90B60
-P 4850 5150
-F 0 "#PWR04" H 4850 4900 50  0001 C CNN
-F 1 "GND" H 4858 4977 50  0000 C CNN
-F 2 "" H 4850 5150 50  0000 C CNN
-F 3 "" H 4850 5150 50  0000 C CNN
-	1    4850 5150
-	1    0    0    -1
-$EndComp
-Wire Wire Line
-	4750 5000 4750 5100
-Wire Wire Line
-	4750 5100 4950 5100
-Wire Wire Line
-	4850 5100 4850 5150
-Wire Wire Line
-	4950 5100 4950 5000
-Connection ~ 4850 5100
-$Comp
-L +5V #PWR05
+L +5V #PWR04
 U 1 1 56E90BE7
 P 6950 3550
-F 0 "#PWR05" H 6950 3400 50  0001 C CNN
+F 0 "#PWR04" H 6950 3400 50  0001 C CNN
 F 1 "+5V" H 6968 3723 50  0000 C CNN
 F 2 "" H 6950 3550 50  0000 C CNN
@@
 	6950 3750 6950 4100
 $Comp
-L GND #PWR06
+L GND #PWR05
 U 1 1 56E90C1C
 P 8200 4200
-F 0 "#PWR06" H 8200 3950 50  0001 C CNN
+F 0 "#PWR05" H 8200 3950 50  0001 C CNN
 F 1 "GND" H 8208 4027 50  0000 C CNN
 F 2 "" H 8200 4200 50  0000 C CNN
@@
 P 6400 4300
 F 0 "D2" V 6354 4378 50  0000 L CNN
-F 1 "LED" V 6445 4378 50  0000 L CNN
+F 1 "TX" V 6445 4378 50  0000 L CNN
 F 2 "LEDs:LED-0603" H 6400 4300 50  0001 C CNN
 F 3 "" H 6400 4300 50  0000 C CNN
@@
 P 6100 4300
 F 0 "D1" V 6054 4378 50  0000 L CNN
-F 1 "LED" V 6145 4378 50  0000 L CNN
+F 1 "RX" V 6145 4378 50  0000 L CNN
 F 2 "LEDs:LED-0603" H 6100 4300 50  0001 C CNN
 F 3 "" H 6100 4300 50  0000 C CNN
@@
 F 0 "R1" H 6170 3896 50  0000 L CNN
 F 1 "R" H 6170 3805 50  0000 L CNN
-F 2 "Resistors_SMD:R_0603" V 6030 3850 50  0001 C CNN
+F 2 "Resistors_SMD:R_0603_HandSoldering" V 6030 3850 50  0001 C CNN
 F 3 "" H 6100 3850 50  0000 C CNN
 	1    6100 3850
@@
 F 0 "R2" H 6470 3896 50  0000 L CNN
 F 1 "R" H 6470 3805 50  0000 L CNN
-F 2 "Resistors_SMD:R_0603" V 6330 3850 50  0001 C CNN
+F 2 "Resistors_SMD:R_0603_HandSoldering" V 6330 3850 50  0001 C CNN
 F 3 "" H 6400 3850 50  0000 C CNN
 	1    6400 3850
@@
 F 0 "C1" H 4665 2946 50  0000 L CNN
 F 1 "C" H 4665 2855 50  0000 L CNN
-F 2 "Capacitors_SMD:C_0603" H 4588 2750 50  0001 C CNN
+F 2 "Capacitors_SMD:C_0603_HandSoldering" H 4588 2750 50  0001 C CNN
 F 3 "" H 4550 2900 50  0000 C CNN
 	1    4550 2900
@@
 Connection ~ 4550 3150
 $Comp
-L GND #PWR07
+L GND #PWR06
 U 1 1 56E9134E
 P 4550 2750
-F 0 "#PWR07" H 4550 2500 50  0001 C CNN
+F 0 "#PWR06" H 4550 2500 50  0001 C CNN
 F 1 "GND" H 4558 2577 50  0000 C CNN
 F 2 "" H 4550 2750 50  0000 C CNN
@@
 	6950 3550 6950 3650
 Wire Wire Line
-	5550 4600 6400 4600
-Wire Wire Line
-	6400 4600 6400 4500
-Wire Wire Line
-	6100 4500 5550 4500
+	6400 4500 6400 5000
 Wire Wire Line
 	6400 4000 6400 4100
@@
 07 00 85 88 3B 00 28 44 DC 01 40 21 E2 0E 00 0A 11 77 00 50 88 B8 03 80 42 C4 1D 00 14 22 EE 00
 A0 10 71 07 00 85 88 3B 00 28 F4 2F 6E 0E 73 66 69 F5 31 42 00 00 00 00 49 45 4E 44 AE 42 60 82
-58
+50
 EndData
 $EndBitmap
+Text Label 5550 4300 0    60   ~ 0
+RST
+Text Label 6950 4400 2    60   ~ 0
+RST
+Wire Wire Line
+	6400 5000 5550 5000
+Wire Wire Line
+	6100 4500 6100 4900
+Wire Wire Line
+	6100 4900 5550 4900
+Wire Wire Line
+	4750 5400 4950 5400
+$Comp
+L GND #PWR07
+U 1 1 57D3D2FC
+P 4850 5450
+F 0 "#PWR07" H 4850 5200 50  0001 C CNN
+F 1 "GND" H 4855 5277 50  0000 C CNN
+F 2 "" H 4850 5450 50  0000 C CNN
+F 3 "" H 4850 5450 50  0000 C CNN
+	1    4850 5450
+	1    0    0    -1
+$EndComp
+Wire Wire Line
+	4850 5450 4850 5400
+Connection ~ 4850 5400
+$Comp
+L LED D3
+U 1 1 57D3DF64
+P 6600 4800
+F 0 "D3" V 6646 4692 50  0000 R CNN
+F 1 "V_TARGET" V 6555 4692 50  0000 R CNN
+F 2 "LEDs:LED-0603" H 6600 4800 50  0001 C CNN
+F 3 "" H 6600 4800 50  0000 C CNN
+	1    6600 4800
+	0    -1   -1   0
+$EndComp
+Wire Wire Line
+	6600 4200 6950 4200
+$Comp
+L R R3
+U 1 1 57D3E0C0
+P 6600 4350
+F 0 "R3" H 6670 4396 50  0000 L CNN
+F 1 "R" H 6670 4305 50  0000 L CNN
+F 2 "Resistors_SMD:R_0603_HandSoldering" V 6530 4350 50  0001 C CNN
+F 3 "" H 6600 4350 50  0000 C CNN
+	1    6600 4350
+	1    0    0    -1
+$EndComp
+$Comp
+L GND #PWR08
+U 1 1 57D3E122
+P 6600 5150
+F 0 "#PWR08" H 6600 4900 50  0001 C CNN
+F 1 "GND" H 6605 4977 50  0000 C CNN
+F 2 "" H 6600 5150 50  0000 C CNN
+F 3 "" H 6600 5150 50  0000 C CNN
+	1    6600 5150
+	1    0    0    -1
+$EndComp
+Wire Wire Line
+	6600 4500 6600 4600
+Wire Wire Line
+	6600 5000 6600 5150
 $EndSCHEMATC

Commit message: Added copper pour to bottom layer
Parts:
- D1, D2, D3: symbol LED -> LED-RESCUE-MysX2USB
- P1: symbol USB_A -> USB_A-RESCUE-MysX2USB
Changed lines of the file:
@@
 EESchema Schematic File Version 2
+LIBS:MysX2USB-rescue
 LIBS:mysensors_sensors
 LIBS:power
@@
 LIBS:mysensors_connectors
 LIBS:MysX2USB-cache
-EELAYER 25 0
+EELAYER 26 0
 EELAYER END
 $Descr A4 11693 8268
@@
 $EndComp
 $Comp
-L USB_A P1
+L USB_A-RESCUE-MysX2USB P1
 U 1 1 56E908FF
 P 3500 4300
@@
 D+
 $Comp
-L LED D2
+L LED-RESCUE-MysX2USB D2
 U 1 1 56E90EFF
 P 6400 4300
@@
 $EndComp
 $Comp
-L LED D1
+L LED-RESCUE-MysX2USB D1
 U 1 1 56E90F3E
 P 6100 4300
@@
 07 00 85 88 3B 00 28 44 DC 01 40 21 E2 0E 00 0A 11 77 00 50 88 B8 03 80 42 C4 1D 00 14 22 EE 00
 A0 10 71 07 00 85 88 3B 00 28 F4 2F 6E 0E 73 66 69 F5 31 42 00 00 00 00 49 45 4E 44 AE 42 60 82
-50
 EndData
 $EndBitmap
@@
 Connection ~ 4850 5400
 $Comp
-L LED D3
+L LED-RESCUE-MysX2USB D3
 U 1 1 57D3DF64
 P 6600 4800
